File: ergo/ergo56.kicad_pcb (KiCad board)
At the start: 2 copper layers, 250.3 x 112.5 mm, 131 parts, among them J1 BAT, J2 AudioJack3_Ground, J3 AudioJack3_Ground, J5 Conn_ARM_SWD, U1 PCA9555PW, U2 Seeeduino Xiao nRF52840

Commit message: stage
Parts:
- removed the REF** at (156.0, 123.2)
- removed the REF** at (140.1, 123.7)
- added REF**: KiCad-Logo2_5mm_SilkScreen, Symbol:KiCad-Logo2_5mm_SilkScreen, F.Cu at (142.8, 92.5)
- added REF**: OSHW-Logo2_7.3x6mm_SilkScreen, Symbol:OSHW-Logo2_7.3x6mm_SilkScreen, F.Cu at (143.4, 56.9)
- J1: moved to B.Cu
- U2: footprint PCM_marbastlib-xp-promicroish:Xiao_nRF52840_ACH -> PCM_marbastlib-xp-promicroish:Xiao_nRF52840_AC_Reflow
- moved H7 299.8 mm to (45.4, 95.5)
- moved H1 266.5 mm to (54.2, 62.7)
- moved H3 220.0 mm to (109.5, 66.6)
- moved H4 215.4 mm to (112.7, 124.6)
- moved H8 163.1 mm to (187.1, 66.6)
- moved H5 154.6 mm to (184.0, 124.6)
- moved R2 89.3 mm to (160.5, 116.5), turned to 15 degrees
- moved R1 88.5 mm to (159.9, 114.5), turned to 15 degrees
- moved H2 87.7 mm to (242.5, 62.7)
- moved H6 85.7 mm to (251.3, 95.6)
- moved J5 84.4 mm to (156.7, 123.2), turned to -90 degrees
- moved J3 68.8 mm to (141.7, 108.0), turned to -105 degrees
- moved U2 68.7 mm to (163.7, 42.2), turned to -75 degrees
- moved C1 67.8 mm to (133.4, 121.0), turned to -90 degrees
- moved U1 64.4 mm to (138.8, 123.2), turned to 90 degrees
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Other:
- board size 250.3 x 112.5 mm -> 250.3 x 117.5 mm
