File: ergo/ergo56.kicad_pcb (KiCad board)
At the start: 2 copper layers, 250.3 x 117.5 mm, 131 parts, among them J1 BAT, J2 AudioJack3_Ground, J3 AudioJack3_Ground, J5 Conn_ARM_SWD, U1 PCA9555PW, U2 Seeeduino Xiao nRF52840

Commit message: fix minor pcb stuff
Routing:
- net GND: vias 46 -> 58
Other:
- board text added: "+"
- board text added: "ergo56 v0.2 202401"
- board text removed: "ergo56 v0.1 202312"
Changed lines of the file:
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@@
   (paper "A4")
   (title_block
-    (date "2023-12-20")
-    (rev "0.1")
+    (date "2024-01-04")
+    (rev "0.2")
     (company "github.com/LDAB")
   )
@@
   (gr_circle (center 187.139552 66.624529) (end 188.789552 66.624529)
     (stroke (width 0.15) (type solid)) (fill none) (layer "User.6"))
-  (gr_text "ergo56 v0.1\n202312" (at 137.41755 127.55753) (layer "B.SilkS")
+  (gr_text "ergo56 v0.2\n202401" (at 137.41755 127.55753) (layer "B.SilkS")
     (effects (font (size 2 2) (thickness 0.35)) (justify mirror))
   )
@@
     (effects (font (size 1.2 1.2) (thickness 0.3)) (justify mirror))
   )
+  (gr_text "+" (at 159.5 128.28) (layer "F.SilkS")
+    (effects (font (size 1 1) (thickness 0.15)) (justify left bottom))
+  )
   (gr_text "github.com/LDAB" (at 153.67355 89.71153 105) (layer "F.SilkS")
     (effects (font (size 1.2 1.2) (thickness 0.3)))
@@
   (segment (start 161.972866 107.96149) (end 166.3728 112.361424) (width 0.25) (layer "B.Cu") (net 6))
   (segment (start 154.000563 139.924532) (end 152.350563 141.574532) (width 0.25) (layer "B.Cu") (net 6))
+  (via (at 138.77 103.37) (size 0.8) (drill 0.4) (layers "F.Cu" "B.Cu") (free) (net 7))
   (via (at 167.4368 60.8076) (size 0.8) (drill 0.4) (layers "F.Cu" "B.Cu") (free) (net 7))
   (via (at 164.7952 114.1476) (size 0.8) (drill 0.4) (layers "F.Cu" "B.Cu") (free) (net 7))
   (via (at 168.6814 117.0432) (size 0.8) (drill 0.4) (layers "F.Cu" "B.Cu") (free) (net 7))
+  (via (at 138.51 126.81) (size 0.8) (drill 0.4) (layers "F.Cu" "B.Cu") (free) (net 7))
   (via (at 110.0582 120.2182) (size 0.8) (drill 0.4) (layers "F.Cu" "B.Cu") (free) (net 7))
   (via (at 175.2346 52.4764) (size 0.8) (drill 0.4) (layers "F.Cu" "B.Cu") (free) (net 7))
   (via (at 162.9664 59.6392) (size 0.8) (drill 0.4) (layers "F.Cu" "B.Cu") (free) (net 7))
+  (via (at 134.84 106.46) (size 0.8) (drill 0.4) (layers "F.Cu" "B.Cu") (free) (net 7))
+  (via (at 145.32 122.23) (size 0.8) (drill 0.4) (layers "F.Cu" "B.Cu") (free) (net 7))
   (via (at 133.6294 96.393) (size 0.8) (drill 0.4) (layers "F.Cu" "B.Cu") (free) (net 7))
   (via (at 148.336 115.316) (size 0.8) (drill 0.4) (layers "F.Cu" "B.Cu") (free) (net 7))
+  (via (at 129.68 112.12) (size 0.8) (drill 0.4) (layers "F.Cu" "B.Cu") (free) (net 7))
+  (via (at 139.5 107.57) (size 0.8) (drill 0.4) (layers "F.Cu" "B.Cu") (free) (net 7))
   (via (at 168.6814 115.5192) (size 0.8) (drill 0.4) (layers "F.Cu" "B.Cu") (free) (net 7))
   (via (at 78.2066 109.1946) (size 0.8) (drill 0.4) (layers "F.Cu" "B.Cu") (free) (net 7))
@@
   (via (at 164.7952 118.618) (size 0.8) (drill 0.4) (layers "F.Cu" "B.Cu") (free) (net 7))
   (via (at 148.5392 69.596) (size 0.8) (drill 0.4) (layers "F.Cu" "B.Cu") (free) (net 7))
+  (via (at 143.54 100.69) (size 0.8) (drill 0.4) (layers "F.Cu" "B.Cu") (free) (net 7))
+  (via (at 132.25 117.12) (size 0.8) (drill 0.4) (layers "F.Cu" "B.Cu") (free) (net 7))
   (via (at 64.6684 110.1852) (size 0.8) (drill 0.4) (layers "F.Cu" "B.Cu") (free) (net 7))
   (via (at 78.4098 98.171) (size 0.8) (drill 0.4) (layers "F.Cu" "B.Cu") (free) (net 7))
@@
   (via (at 154.8384 68.2244) (size 0.8) (drill 0.4) (layers "F.Cu" "B.Cu") (free) (net 7))
   (via (at 133.5532 100.1268) (size 0.8) (drill 0.4) (layers "F.Cu" "B.Cu") (free) (net 7))
+  (via (at 141.72 112.42) (size 0.8) (drill 0.4) (layers "F.Cu" "B.Cu") (free) (net 7))
   (via (at 148.336 113.792) (size 0.8) (drill 0.4) (layers "F.Cu" "B.Cu") (free) (net 7))
   (via (at 99.4664 103.8098) (size 0.8) (drill 0.4) (layers "F.Cu" "B.Cu") (free) (net 7))
@@
   (via (at 153.3652 57.0992) (size 0.8) (drill 0.4) (layers "F.Cu" "B.Cu") (free) (net 7))
   (via (at 152.019 129.413) (size 0.8) (drill 0.4) (layers "F.Cu" "B.Cu") (free) (net 7))
+  (via (at 143.05 107.28) (size 0.8) (drill 0.4) (layers "F.Cu" "B.Cu") (free) (net 7))
   (via (at 168.3512 42.7736) (size 0.8) (drill 0.4) (layers "F.Cu" "B.Cu") (free) (net 7))
+  (via (at 145.45 114.63) (size 0.8) (drill 0.4) (layers "F.Cu" "B.Cu") (free) (net 7))
   (via (at 167.4622 45.72) (size 0.8) (drill 0.4) (layers "F.Cu" "B.Cu") (free) (net 7))
   (via (at 116.2812 112.6236) (size 0.8) (drill 0.4) (layers "F.Cu" "B.Cu") (free) (net 7))
@@
   (via (at 176.8348 50.8762) (size 0.8) (drill 0.4) (layers "F.Cu" "B.Cu") (free) (net 7))
   (via (at 148.336 118.364) (size 0.8) (drill 0.4) (layers "F.Cu" "B.Cu") (free) (net 7))
+  (via (at 137.5 109.91) (size 0.8) (drill 0.4) (layers "F.Cu" "B.Cu") (free) (net 7))
   (via (at 165.989 43.3324) (size 0.8) (drill 0.4) (layers "F.Cu" "B.Cu") (free) (net 7))
   (via (at 165.5318 39.8018) (size 0.8) (drill 0.4) (layers "F.Cu" "B.Cu") (free) (net 7))
