File: basic/basic60.kicad_pcb (KiCad board)
At the start: 2 copper layers, 250.3 x 117.5 mm, 131 parts, among them J1 BAT, J2 AudioJack3_Ground, J3 AudioJack3_Ground, J5 Conn_ARM_SWD, U1 PCA9555PW, U2 Seeeduino Xiao nRF52840

Commit message: basic60
Parts:
- added D49: ~, Diode_SMD:D_SOD-123, F.Cu at (51.2, 124.8)
- added D50: ~, Diode_SMD:D_SOD-123, F.Cu at (69.2, 124.8)
- added D59: ~, Diode_SMD:D_SOD-123, F.Cu at (231.2, 124.8)
- added D60: ~, Diode_SMD:D_SOD-123, F.Cu at (249.2, 124.8)
- added SW49: SW_Push, PCM_marbastlib-choc:SW_choc_v1_HS_1u, B.Cu at (51.2, 120.2)
- added SW50: SW_Push, PCM_marbastlib-choc:SW_choc_v1_HS_1u, B.Cu at (69.2, 120.2)
- added SW59: SW_Push, PCM_marbastlib-choc:SW_choc_v1_HS_1u, B.Cu at (231.2, 120.2)
- added SW60: SW_Push, PCM_marbastlib-choc:SW_choc_v1_HS_1u, B.Cu at (249.2, 120.2)
- J1: renamed from J5; value Conn_ARM_SWD -> Conn_ARM_SW
- moved U1 250.9 mm to (-43.9, 183.1)
- moved SW48 214.5 mm to (249.2, 103.2), turned to 0 degrees
- moved D48 213.6 mm to (249.2, 107.8), turned to 180 degrees
- moved SW37 210.7 mm to (51.2, 103.2), turned to 0 degrees
- moved SW36 210.1 mm to (249.2, 86.2), turned to 0 degrees
- moved D37 209.7 mm to (51.2, 107.8), turned to 180 degrees
- moved D36 209.1 mm to (249.2, 90.8), turned to 180 degrees
- moved SW25 206.3 mm to (51.2, 86.2), turned to 0 degrees
- moved SW24 205.7 mm to (249.2, 69.2), turned to 0 degrees
- moved D25 205.3 mm to (51.2, 90.8), turned to 180 degrees
- moved D24 204.7 mm to (249.2, 73.8), turned to 180 degrees
- moved SW13 201.9 mm to (51.2, 69.2), turned to 0 degrees
- moved SW12 201.3 mm to (249.2, 52.2), turned to 0 degrees
- moved D13 200.9 mm to (51.2, 73.8), turned to 180 degrees
- moved D12 200.3 mm to (249.2, 56.8), turned to 180 degrees
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- renumbered D_A6 to D1, D_B9 to D10, D_B10 to D11, D_B11 to D12, D_A0 to D13, D_A1 to D14, D_A2 to D15, D_A3 to D16, D_A4 to D17, D_A5 to D18, D_B0 to D19, D_A7 to D2, D_B1 to D20, D_B2 to D21, D_B3 to D22, D_B4 to D23, D_B5 to D24, D_C0 to D25, D_C1 to D26, D_C2 to D27, D_C3 to D28, D_C4 to D29, D_A8 to D3, D_C5 to D30, D_D0 to D31, D_D1 to D32, D_D2 to D33, D_D3 to D34, D_D4 to D35, D_D5 to D36, D_E0 to D37, D_E1 to D38, D_E2 to D39, D_A9 to D4, D_E3 to D40, D_E4 to D41, D_E5 to D42, D_F0 to D43, D_F1 to D44, D_F2 to D45, D_F3 to D46, D_F4 to D47, D_F5 to D48, D_A10 to D5, D_G0 to D51, D_G1 to D52, D_G2 to D53, D_G3 to D54, D_G4 to D55, D_G6 to D56, D_G7 to D57, D_G8 to D58, D_A11 to D6, D_B6 to D7, D_B7 to D8, D_B8 to D9, H2 to H1, H3 to H2, H1 to H3, H7 to H6, H6 to H7, J3 to J2, J2 to J3, J1 to J4, SwA6 to SW1, SwB9 to SW10, SwB10 to SW11, SwB11 to SW12, SwA0 to SW13, SwA1 to SW14, SwA2 to SW15, SwA3 to SW16, SwA4 to SW17, SwA5 to SW18, SwB0 to SW19, SwA7 to SW2, SwB1 to SW20, SwB2 to SW21, SwB3 to SW22, SwB4 to SW23, SwB5 to SW24, SwC0 to SW25, SwC1 to SW26, SwC2 to SW27, SwC3 to SW28, SwC4 to SW29, SwA8 to SW3, SwC5 to SW30, SwD0 to SW31, SwD1 to SW32, SwD2 to SW33, SwD3 to SW34, SwD4 to SW35, SwD5 to SW36, SwE0 to SW37, SwE1 to SW38, SwE2 to SW39, SwA9 to SW4, SwE3 to SW40, SwE4 to SW41, SwE5 to SW42, SwF0 to SW43, SwF1 to SW44, SwF2 to SW45, SwF3 to SW46, SwF4 to SW47, SwF5 to SW48, SwA10 to SW5, SwG0 to SW51, SwG1 to SW52, SwG2 to SW53, SwG3 to SW54, SwG4 to SW55, SwG6 to SW56, SwG7 to SW57, SwG8 to SW58, SwA11 to SW6, SwB6 to SW7, SwB7 to SW8, SwB8 to SW9, U2 to U1, U1 to U2
Connections:
- net SWDCLK renamed SWCLK
- net SWDIO renamed SWIO
Routing:
- net col5: track 108.4 -> 680.0 mm, vias 1 -> 0
- net col4: track 113.1 -> 680.0 mm, vias 1 -> 0
- net col7: track 117.8 -> 680.0 mm, vias 1 -> 0
- net col2: track 125.5 -> 680.0 mm, vias 1 -> 0
- net col8: track 143.4 -> 680.0 mm, vias 1 -> 0
- net col9: track 158.3 -> 663.0 mm
- net col1: track 119.5 -> 595.0 mm, vias 1 -> 0
- net col11: track 173.2 -> 595.0 mm, vias 1 -> 0
- net col6: track 97.2 -> 510.0 mm, vias 1 -> 0
- net col3: track 115.0 -> 510.0 mm, vias 1 -> 0
- net col0: track 138.0 -> 425.0 mm, vias 1 -> 0
- net col10: track 155.5 -> 425.0 mm
- net +3V3: track 169.9 -> 0.00 mm, vias 2 -> 0
- net SCL: track 126.4 -> 0.00 mm, vias 4 -> 0
- net SDA: track 118.8 -> 0.00 mm, vias 4 -> 0
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Other:
- board size 250.3 x 117.5 mm -> 216 x 85 mm
- board text added: "basic60 v0.1 202312"
- board text removed: "ergo56 v0.1 202312"

Commit message: finish pcb
Parts:
- J1: moved to B.Cu
- moved U1 260.3 mm to (172.6, 38.7), turned to -90 degrees
- moved J4 241.3 mm to (173.8, 32.6), turned to 180 degrees
- moved J1 232.5 mm to (164.3, 34.0), turned to 0 degrees
- moved J2 217.7 mm to (144.2, 39.8), turned to -90 degrees
- moved J3 216.7 mm to (156.4, 39.7), turned to -90 degrees
- moved U2 213.4 mm to (127.3, 39.6)
- moved C1 213.3 mm to (129.4, 34.5)
- moved R2 213.0 mm to (156.7, 46.5), turned to 0 degrees
- moved R1 211.8 mm to (156.7, 48.0), turned to 0 degrees
- moved REF** 191.1 mm to (126.7, 46.9), turned to 0 degrees
- moved REF** 80.3 mm to (127.2, 30.4)
- moved D49 6.31 mm to (51.2, 131.1)
- moved D50 6.31 mm to (69.2, 131.1)
- moved D51 6.31 mm to (87.2, 131.1)
- moved D52 6.31 mm to (105.2, 131.1)
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Connections:
- D1 pad 1: row0 -> row5
- D10 pad 1: row5 -> row0
- D11 pad 1: row5 -> row0
- D12 pad 1: row5 -> row0
- D13 pad 1: row1 -> row6
- D14 pad 1: row1 -> row6
- D15 pad 1: row1 -> row6
- D16 pad 1: row1 -> row6
- D17 pad 1: row1 -> row6
- D18 pad 1: row1 -> row6
- D19 pad 1: row6 -> row1
- D2 pad 1: row0 -> row5
- D20 pad 1: row6 -> row1
- D21 pad 1: row6 -> row1
- D22 pad 1: row6 -> row1
- D23 pad 1: row6 -> row1
- D24 pad 1: row6 -> row1
- D25 pad 1: row2 -> row7
- D26 pad 1: row2 -> row7
- D27 pad 1: row2 -> row7
- D28 pad 1: row2 -> row7
- D29 pad 1: row2 -> row7
- D3 pad 1: row0 -> row5
- D30 pad 1: row2 -> row7
- D31 pad 1: row7 -> row2
- D32 pad 1: row7 -> row2
- D33 pad 1: row7 -> row2
- D34 pad 1: row7 -> row2
- D35 pad 1: row7 -> row2
- D36 pad 1: row7 -> row2
- D37 pad 1: row3 -> row8
- D38 pad 1: row3 -> row8
- D39 pad 1: row3 -> row8
- D4 pad 1: row0 -> row5
- D40 pad 1: row3 -> row8
- D41 pad 1: row3 -> row8
- D42 pad 1: row3 -> row8
- D43 pad 1: row8 -> row3
- D44 pad 1: row8 -> row3
- D45 pad 1: row8 -> row3
- D46 pad 1: row8 -> row3
- D47 pad 1: row8 -> row3
- D48 pad 1: row8 -> row3
- D49 pad 1: row4 -> row9
- D5 pad 1: row0 -> row5
- D50 pad 1: row4 -> row9
- D51 pad 1: row4 -> row9
- D52 pad 1: row4 -> row9
- D53 pad 1: row4 -> row9
- D54 pad 1: row4 -> row9
- D55 pad 1: row9 -> row4
- D56 pad 1: row9 -> row4
- D57 pad 1: row9 -> row4
- D58 pad 1: row9 -> row4
- D59 pad 1: row9 -> row4
- D6 pad 1: row0 -> row5
- D60 pad 1: row9 -> row4
- D7 pad 1: row5 -> row0
- D8 pad 1: row5 -> row0
- D9 pad 1: row5 -> row0
- SW1 pad 1: col0 -> col11
- SW10 pad 1: col9 -> col2
- SW11 pad 1: col10 -> col1
- SW12 pad 1: col11 -> col0
- SW13 pad 1: col0 -> col11
- SW14 pad 1: col1 -> col10
- SW15 pad 1: col2 -> col9
- SW16 pad 1: col3 -> col8
- SW17 pad 1: col4 -> col7
- SW18 pad 1: col5 -> col6
- SW19 pad 1: col6 -> col5
- SW2 pad 1: col1 -> col10
- SW20 pad 1: col7 -> col4
- SW21 pad 1: col8 -> col3
- SW22 pad 1: col9 -> col2
- SW23 pad 1: col10 -> col1
- SW24 pad 1: col11 -> col0
- SW25 pad 1: col0 -> col11
- SW26 pad 1: col1 -> col10
- SW27 pad 1: col2 -> col9
- SW28 pad 1: col3 -> col8
- SW29 pad 1: col4 -> col7
- SW3 pad 1: col2 -> col9
- SW30 pad 1: col5 -> col6
- SW31 pad 1: col6 -> col5
- SW32 pad 1: col7 -> col4
- SW33 pad 1: col8 -> col3
- SW34 pad 1: col9 -> col2
- SW35 pad 1: col10 -> col1
- SW36 pad 1: col11 -> col0
- SW37 pad 1: col0 -> col11
- SW38 pad 1: col1 -> col10
- SW39 pad 1: col2 -> col9
- SW4 pad 1: col3 -> col8
- SW40 pad 1: col3 -> col8
- SW41 pad 1: col4 -> col7
- SW42 pad 1: col5 -> col6
- SW43 pad 1: col6 -> col5
- SW44 pad 1: col7 -> col4
- SW45 pad 1: col8 -> col3
- SW46 pad 1: col9 -> col2
- SW47 pad 1: col10 -> col1
- SW48 pad 1: col11 -> col0
- SW49 pad 1: col0 -> col11
- SW5 pad 1: col4 -> col7
- SW50 pad 1: col1 -> col10
- SW51 pad 1: col2 -> col9
- SW52 pad 1: col3 -> col8
- SW53 pad 1: col4 -> col7
- SW54 pad 1: col5 -> col6
- SW55 pad 1: col6 -> col5
- SW56 pad 1: col7 -> col4
- SW57 pad 1: col8 -> col3
- SW58 pad 1: col9 -> col2
- SW59 pad 1: col10 -> col1
- SW6 pad 1: col5 -> col6
- SW60 pad 1: col11 -> col0
- SW7 pad 1: col6 -> col5
- SW8 pad 1: col7 -> col4
- SW9 pad 1: col8 -> col3
Routing:
- net col5: track 680.0 -> 84.1 mm
- net col7: track 680.0 -> 84.6 mm
- net col8: track 680.0 -> 90.9 mm
- net col4: track 680.0 -> 95.0 mm, vias 0 -> 1
- net col9: track 663.0 -> 105.6 mm, vias 0 -> 1
- net col2: track 680.0 -> 127.1 mm, vias 0 -> 1
- net col1: track 595.0 -> 140.7 mm, vias 0 -> 1
- net col11: track 595.0 -> 146.1 mm
- net col6: track 510.0 -> 100.7 mm, vias 0 -> 1
- net col3: track 510.0 -> 111.0 mm, vias 0 -> 1
- net col10: track 425.0 -> 124.9 mm, vias 0 -> 1
- net col0: track 425.0 -> 152.8 mm
- net row4: track 93.8 -> 210.4 mm, vias 0 -> 2
- net row9: track 93.8 -> 196.6 mm
- net row3: track 93.8 -> 196.4 mm, vias 0 -> 2
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Other:
- board size 216 x 85 mm -> 216 x 108.2 mm
