File: basic/basic60.kicad_sch (KiCad schematic)
At the start: 129 parts, among them J1 BAT, J2 AudioJack3_Ground, J3 AudioJack3_Ground, J5 Conn_ARM_SWD, U1 PCA9555PW, U2 Seeeduino Xiao nRF52840

Commit message: basic60
Parts:
- added D49, D50, D59, D60: ~, Diode_SMD:D_SOD-123, symbol Diode:1N4148W
- added SW49, SW50, SW59, SW60: SW_Push, PCM_marbastlib-choc:SW_choc_v1_HS_1u, symbol Switch:SW_Push
- J1: renamed from J5; value Conn_ARM_SWD -> Conn_ARM_SW
- renumbered D_A6 to D1, D_B9 to D10, D_B10 to D11, D_B11 to D12, D_A0 to D13, D_A1 to D14, D_A2 to D15, D_A3 to D16, D_A4 to D17, D_A5 to D18, D_B0 to D19, D_A7 to D2, D_B1 to D20, D_B2 to D21, D_B3 to D22, D_B4 to D23, D_B5 to D24, D_C0 to D25, D_C1 to D26, D_C2 to D27, D_C3 to D28, D_C4 to D29, D_A8 to D3, D_C5 to D30, D_D0 to D31, D_D1 to D32, D_D2 to D33, D_D3 to D34, D_D4 to D35, D_D5 to D36, D_E0 to D37, D_E1 to D38, D_E2 to D39, D_A9 to D4, D_E3 to D40, D_E4 to D41, D_E5 to D42, D_F0 to D43, D_F1 to D44, D_F2 to D45, D_F3 to D46, D_F4 to D47, D_F5 to D48, D_A10 to D5, D_G0 to D51, D_G1 to D52, D_G2 to D53, D_G3 to D54, D_G4 to D55, D_G6 to D56, D_G7 to D57, D_G8 to D58, D_A11 to D6, D_B6 to D7, D_B7 to D8, D_B8 to D9, H2 to H1, H3 to H2, H1 to H3, H7 to H6, H6 to H7, J3 to J2, J2 to J3, J1 to J4, SwA6 to SW1, SwB9 to SW10, SwB10 to SW11, SwB11 to SW12, SwA0 to SW13, SwA1 to SW14, SwA2 to SW15, SwA3 to SW16, SwA4 to SW17, SwA5 to SW18, SwB0 to SW19, SwA7 to SW2, SwB1 to SW20, SwB2 to SW21, SwB3 to SW22, SwB4 to SW23, SwB5 to SW24, SwC0 to SW25, SwC1 to SW26, SwC2 to SW27, SwC3 to SW28, SwC4 to SW29, SwA8 to SW3, SwC5 to SW30, SwD0 to SW31, SwD1 to SW32, SwD2 to SW33, SwD3 to SW34, SwD4 to SW35, SwD5 to SW36, SwE0 to SW37, SwE1 to SW38, SwE2 to SW39, SwA9 to SW4, SwE3 to SW40, SwE4 to SW41, SwE5 to SW42, SwF0 to SW43, SwF1 to SW44, SwF2 to SW45, SwF3 to SW46, SwF4 to SW47, SwF5 to SW48, SwA10 to SW5, SwG0 to SW51, SwG1 to SW52, SwG2 to SW53, SwG3 to SW54, SwG4 to SW55, SwG6 to SW56, SwG7 to SW57, SwG8 to SW58, SwA11 to SW6, SwB6 to SW7, SwB7 to SW8, SwB8 to SW9, U2 to U1, U1 to U2
Connections:
- net col0: now also SW49.1
- net col1: now also SW50.1
- net col10: now also SW59.1
- net col11: now also SW60.1
- net row4: now also D49.1 (K), D50.1 (K)
- net row9: now also D59.1 (K), D60.1 (K)
- net SWDCLK renamed SWCLK
- net SWDIO renamed SWIO
- new net: D49.2 (A), SW49.2
- new net: D50.2 (A), SW50.2
- new net: D60.2 (A), SW60.2
- new net: D59.2 (A), SW59.2
Other:
- title: ergo56 -> basic60

Commit message: finish pcb
Parts:
- renumbered D7 to D1, D4 to D10, D5 to D11, D6 to D12, D19 to D13, D20 to D14, D21 to D15, D22 to D16, D23 to D17, D24 to D18, D13 to D19, D8 to D2, D14 to D20, D15 to D21, D16 to D22, D17 to D23, D18 to D24, D31 to D25, D32 to D26, D33 to D27, D34 to D28, D35 to D29, D9 to D3, D36 to D30, D25 to D31, D26 to D32, D27 to D33, D28 to D34, D29 to D35, D30 to D36, D43 to D37, D44 to D38, D45 to D39, D10 to D4, D46 to D40, D47 to D41, D48 to D42, D37 to D43, D38 to D44, D39 to D45, D40 to D46, D41 to D47, D42 to D48, D55 to D49, D11 to D5, D56 to D50, D57 to D51, D58 to D52, D59 to D53, D60 to D54, D49 to D55, D50 to D56, D51 to D57, D52 to D58, D53 to D59, D12 to D6, D54 to D60, D1 to D7, D2 to D8, D3 to D9, SW7 to SW1, SW4 to SW10, SW5 to SW11, SW6 to SW12, SW19 to SW13, SW20 to SW14, SW21 to SW15, SW22 to SW16, SW23 to SW17, SW24 to SW18, SW13 to SW19, SW8 to SW2, SW14 to SW20, SW15 to SW21, SW16 to SW22, SW17 to SW23, SW18 to SW24, SW31 to SW25, SW32 to SW26, SW33 to SW27, SW34 to SW28, SW35 to SW29, SW9 to SW3, SW36 to SW30, SW25 to SW31, SW26 to SW32, SW27 to SW33, SW28 to SW34, SW29 to SW35, SW30 to SW36, SW43 to SW37, SW44 to SW38, SW45 to SW39, SW10 to SW4, SW46 to SW40, SW47 to SW41, SW48 to SW42, SW37 to SW43, SW38 to SW44, SW39 to SW45, SW40 to SW46, SW41 to SW47, SW42 to SW48, SW55 to SW49, SW11 to SW5, SW56 to SW50, SW57 to SW51, SW58 to SW52, SW59 to SW53, SW60 to SW54, SW49 to SW55, SW50 to SW56, SW51 to SW57, SW52 to SW58, SW53 to SW59, SW12 to SW6, SW54 to SW60, SW1 to SW7, SW2 to SW8, SW3 to SW9
Connections:
- net col0: now also SW12.1, SW24.1, SW36.1, SW48.1, SW60.1; no longer SW19.1, SW31.1, SW43.1, SW55.1, SW7.1
- net col1: now also SW11.1, SW23.1, SW35.1, SW47.1, SW59.1; no longer SW20.1, SW32.1, SW44.1, SW56.1, SW8.1
- net col10: now also SW14.1, SW2.1, SW26.1, SW38.1, SW50.1; no longer SW17.1, SW29.1, SW41.1, SW5.1, SW53.1
- net col11: now also SW1.1, SW13.1, SW25.1, SW37.1, SW49.1; no longer SW18.1, SW30.1, SW42.1, SW54.1, SW6.1
- net col2: now also SW10.1, SW22.1, SW34.1, SW46.1, SW58.1; no longer SW21.1, SW33.1, SW45.1, SW57.1, SW9.1
- net col3: now also SW21.1, SW33.1, SW45.1, SW57.1, SW9.1; no longer SW10.1, SW22.1, SW34.1, SW46.1, SW58.1
- net col4: now also SW20.1, SW32.1, SW44.1, SW56.1, SW8.1; no longer SW11.1, SW23.1, SW35.1, SW47.1, SW59.1
- net col5: now also SW19.1, SW31.1, SW43.1, SW55.1, SW7.1; no longer SW12.1, SW24.1, SW36.1, SW48.1, SW60.1
- net col6: now also SW18.1, SW30.1, SW42.1, SW54.1, SW6.1; no longer SW1.1, SW13.1, SW25.1, SW37.1, SW49.1
- net col7: now also SW17.1, SW29.1, SW41.1, SW5.1, SW53.1; no longer SW14.1, SW2.1, SW26.1, SW38.1, SW50.1
- net col8: now also SW16.1, SW28.1, SW4.1, SW40.1, SW52.1; no longer SW15.1, SW27.1, SW3.1, SW39.1, SW51.1
- net col9: now also SW15.1, SW27.1, SW3.1, SW39.1, SW51.1; no longer SW16.1, SW28.1, SW4.1, SW40.1, SW52.1
Other:
- moved on the sheet: D1, D10, D11, D12, D13, D14, D15, D16, D17, D18, D19, D2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
